Commit message: Maze Slam

File: AMR_ws/src/custom_bot/urdf/bot.urdf (robot description, URDF)
Before this commit: robot diff_drive_bot, 6 links, 5 joints
Joints:
- joint base_link_to_left_wheel: axis 0 0 -1  -> 0 0 1 
- joint base_link_to_right_wheel: axis 0 0 1  -> 0 0 -1 

File: AMR_ws/src/custom_bot/urdf/diff_drive_bot.xacro (robot description, xacro)
@@ -127,6 +127,6 @@
     </link>
     <link name="sensor_laser">
-        <visual>
-            <origin rpy="0 0 0" xyz="0 0 0"/>
+        <origin rpy="0 0 3.14159" xyz="0 0 0"/>
+        <visual>
             <geometry>
                 <cylinder radius="${laser_radius}" length="${laser_height}"/>
@@ -139,7 +139,6 @@
         </inertial>
         <collision>
-            <origin rpy="0 0 0" xyz="0 0 0.0125"/>
-            <geometry>
-                <cylinder radius="${laser_radius}" length="${laser_height}"/>
+            <geometry>
+                <cylinder radius="${laser_radius - 0.001}" length="${laser_height- 0.001}"/>
             </geometry>
         </collision>
@@ -158,5 +157,5 @@
         </inertial>
         <collision>
-            <origin rpy="0 0 0" xyz="0 0 0.0125"/>
+            <origin rpy="0 0 0" xyz="0 0 0"/>
             <geometry>
                 <box size="${camera_dim}"/>
@@ -180,11 +179,11 @@
     </joint>
     <joint name="base_link_to_right_wheel" type="continuous">
+        <origin rpy="-1.57079632679 0  0 " xyz="0.0267 -0.13 -0.02"/>
+        <axis xyz="0 0 1 "/>
+        <parent link="base_link"/>
+        <child link="right_wheel"/>
+    </joint>
+    <joint name="base_link_to_left_wheel" type="continuous">
         <origin rpy="1.57079632679 0  0 " xyz="0.0267 0.13 -0.02"/>
-        <axis xyz="0 0 1 "/>
-        <parent link="base_link"/>
-        <child link="right_wheel"/>
-    </joint>
-    <joint name="base_link_to_left_wheel" type="continuous">
-        <origin rpy="-1.57079632679 0  0 " xyz="0.0267 -0.13 -0.02"/>
         <axis xyz="0 0 -1 "/>
         <parent link="base_link"/>
@@ -192,5 +191,5 @@
     </joint>
     <joint name="base_link_to_laser" type="fixed">
-        <origin rpy="0 0  0 " xyz="0.0 0.0 ${laser_height/2}"/>
+        <origin rpy="0 0 0 " xyz="-0.05 0.0 ${0.005 + laser_height/2}"/>
         <axis xyz="0 0 0 "/>
         <parent link="base_link"/>
@@ -198,5 +197,5 @@
     </joint>
     <joint name="base_link_to_camera" type="fixed">
-        <origin rpy="0 0 ${pi_rads}" xyz="-0.08 0.0 0.0"/>
+        <origin rpy="0 0 0" xyz="0.09 0.0 0.0"/>
         <axis xyz="0 0 0 "/>
         <parent link="base_link"/>

File: AMR_ws/src/custom_bot/urdf/gazebo.xacro (robot description, xacro)
@@ -46,6 +46,6 @@
                             <samples>720</samples>
                             <resolution>1</resolution>
-                            <min_angle>-1.570796</min_angle>
-                            <max_angle>1.570796</max_angle>
+                            <min_angle>-1.5708</min_angle>
+                            <max_angle>1.5708</max_angle>
                         </horizontal>
                     </scan>

Commit message: ..

File: AMR_ws/src/custom_bot/urdf/bot.urdf (robot description, URDF)
Before this commit: robot diff_drive_bot, 6 links, 5 joints
Joints:
- joint base_link_to_left_wheel: axis 0 0 1  -> 0 0 -1 
- joint base_link_to_right_wheel: axis 0 0 -1  -> 0 0 1 

File: AMR_ws/src/custom_bot/urdf/diff_drive_bot.xacro (robot description, xacro)
@@ -127,6 +127,6 @@
     </link>
     <link name="sensor_laser">
-        <origin rpy="0 0 3.14159" xyz="0 0 0"/>
-        <visual>
+        <visual>
+            <origin rpy="0 0 0" xyz="0 0 0"/>
             <geometry>
                 <cylinder radius="${laser_radius}" length="${laser_height}"/>
@@ -139,6 +139,7 @@
         </inertial>
         <collision>
-            <geometry>
-                <cylinder radius="${laser_radius - 0.001}" length="${laser_height- 0.001}"/>
+            <origin rpy="0 0 0" xyz="0 0 0.0125"/>
+            <geometry>
+                <cylinder radius="${laser_radius}" length="${laser_height}"/>
             </geometry>
         </collision>
@@ -157,5 +158,5 @@
         </inertial>
         <collision>
-            <origin rpy="0 0 0" xyz="0 0 0"/>
+            <origin rpy="0 0 0" xyz="0 0 0.0125"/>
             <geometry>
                 <box size="${camera_dim}"/>
@@ -179,11 +180,11 @@
     </joint>
     <joint name="base_link_to_right_wheel" type="continuous">
+        <origin rpy="1.57079632679 0  0 " xyz="0.0267 0.13 -0.02"/>
+        <axis xyz="0 0 1 "/>
+        <parent link="base_link"/>
+        <child link="right_wheel"/>
+    </joint>
+    <joint name="base_link_to_left_wheel" type="continuous">
         <origin rpy="-1.57079632679 0  0 " xyz="0.0267 -0.13 -0.02"/>
-        <axis xyz="0 0 1 "/>
-        <parent link="base_link"/>
-        <child link="right_wheel"/>
-    </joint>
-    <joint name="base_link_to_left_wheel" type="continuous">
-        <origin rpy="1.57079632679 0  0 " xyz="0.0267 0.13 -0.02"/>
         <axis xyz="0 0 -1 "/>
         <parent link="base_link"/>
@@ -191,5 +192,5 @@
     </joint>
     <joint name="base_link_to_laser" type="fixed">
-        <origin rpy="0 0 0 " xyz="-0.05 0.0 ${0.005 + laser_height/2}"/>
+        <origin rpy="0 0  0 " xyz="0.0 0.0 ${laser_height/2}"/>
         <axis xyz="0 0 0 "/>
         <parent link="base_link"/>
@@ -197,5 +198,5 @@
     </joint>
     <joint name="base_link_to_camera" type="fixed">
-        <origin rpy="0 0 0" xyz="0.09 0.0 0.0"/>
+        <origin rpy="0 0 ${pi_rads}" xyz="-0.08 0.0 0.0"/>
         <axis xyz="0 0 0 "/>
         <parent link="base_link"/>

File: AMR_ws/src/custom_bot/urdf/gazebo.xacro (robot description, xacro)
@@ -46,6 +46,6 @@
                             <samples>720</samples>
                             <resolution>1</resolution>
-                            <min_angle>-1.5708</min_angle>
-                            <max_angle>1.5708</max_angle>
+                            <min_angle>-1.570796</min_angle>
+                            <max_angle>1.570796</max_angle>
                         </horizontal>
                     </scan>
