Commit message: xacro properties added

File: AMR_ws/src/custom_bot/urdf/diff_drive_bot.xacro (robot description, xacro)
@@ -1,24 +1,13 @@
 <?xml version="1.0"?>
-<!--Autonomous Robots-->
-<!--URDF Mesh-->
+<!--Differential Drive Robot Definition-->
 <!--Author: Sreejith S-->
-<!--Date: Mon 27 Apr 2020 14:39:24 UTC-->
-<robot name="diff_drive_bot">
-    <!--Materials color predefined-->
-  <material name="black">
-    <color rgba="0.0 0.0 0.0 1.0"/>
-  </material>
-  <material name="blue">
-    <color rgba="0 0 0.8 1.0"/>
-  </material>
-  <material name="green">
-    <color rgba="0.0 0.8 0.0 1.0"/>
-  </material>
-  <material name="red">
-    <color rgba="1.0 0 0 1.0"/>
-  </material>
-  <material name="white">
-    <color rgba="1.0 1.0 1.0 1.0"/>
-  </material>
+<!--Date: Fri 15 May 2020 17:26:48 UTC-->
+<robot name="diff_drive_bot" xmlns:xacro="http://www.ros.org/wiki/xacro">
+    <!--Materials-->
+    <xacro:include filename="$(find custom_bot)/urdf/materials.xacro"/>
+    <xacro:include filename="$(find custom_bot)/urdf/gazebo.xacro"/>
+    <!--Properties-->
+    <xacro:property name="wheel_radius" value="4.4"/>
+    <xacro:property name="wheel_width" value="2.4"/>
   <link name="base_footprint">
     <!--<inertial>-->

Commit message: Add laser scanner

File: AMR_ws/src/custom_bot/urdf/diff_drive_bot.xacro (robot description, xacro)
@@ -8,12 +8,15 @@
     <xacro:include filename="$(find custom_bot)/urdf/gazebo.xacro"/>
     <!--Properties-->
-    <xacro:property name="wheel_radius" value="4.4"/>
-    <xacro:property name="wheel_width" value="2.4"/>
+    <xacro:property name="wheel_radius" value="0.032"/>
+    <xacro:property name="wheel_width" value="0.025"/>
+    <xacro:property name="laser_radius" value="0.025"/>
+    <xacro:property name="laser_height" value="0.025"/>
+    <!--Macros-->
+    <xacro:macro name="cylinder_inertia" params="mass r l">
+        <inertia ixx="${mass*(3*r*r+l*l)/12}" ixy="0" ixz="0"
+            iyy="${mass*(3*r*r+l*l)/12}" iyz="0.0"
+            izz="${mass*(r*r)/2}"/>
+    </xacro:macro>
   <link name="base_footprint">
-    <!--<inertial>-->
-      <!--<mass value="0.0001"/>-->
-      <!--<origin xyz="0 0 0"/>-->
-      <!--<inertia ixx="0.0" ixy="0.0" ixz="0.0" iyy="0.0" iyz="0.0" izz="0.0"/>-->
-    <!--</inertial>-->
     <visual>
       <origin rpy="0 0 0" xyz="0 0 0"/>
@@ -97,5 +100,5 @@
             <origin rpy="0 0 0" xyz="0 0 0.0125"/>
             <geometry>
-                <cylinder radius="0.032" length="0.025"/>
+                <cylinder radius="${wheel_radius}" length="${wheel_width}"/>
             </geometry>
         </collision>
@@ -117,5 +120,24 @@
             <origin rpy="0 0 0" xyz="0 0 0.0125"/>
             <geometry>
-                <cylinder radius="0.032" length="0.025"/>
+                <cylinder radius="${wheel_radius}" length="${wheel_width}"/>
+            </geometry>
+        </collision>
+    </link>
+    <link name="sensor_laser">
+        <visual>
+            <origin rpy="0 0 0" xyz="0 0 0"/>
+            <geometry>
+                <cylinder radius="${laser_radius}" length="${laser_height}"/>
+            </geometry>
+            <material name="yellow"/>
+        </visual>
+        <inertial>
+            <mass value="1"/>
+            <xacro:cylinder_inertia mass="1" r="${laser_radius}" l="${laser_height}"/>
+        </inertial>
+        <collision>
+            <origin rpy="0 0 0" xyz="0 0 0.0125"/>
+            <geometry>
+                <cylinder radius="${laser_radius}" length="${laser_height}"/>
             </geometry>
         </collision>
@@ -148,3 +170,9 @@
         <child link="left_wheel"/>
     </joint>
+    <joint name="base_link_to_laser" type="fixed">
+        <origin rpy="0 0  0 " xyz="0.0 0.0 ${laser_height/2}"/>
+        <axis xyz="0 0 0 "/>
+        <parent link="base_link"/>
+        <child link="sensor_laser"/>
+    </joint>
 </robot>

File: AMR_ws/src/custom_bot/urdf/gazebo.xacro (robot description, xacro)
@@ -6,4 +6,5 @@
     <!--If the <gazebo> tag is used without reference property, it is assumed-->
     <!--the element is for the entire robot-->
+    <!--Materials-->
     <gazebo reference="base_link">
         <material>Gazebo/Orange</material>
@@ -14,4 +15,7 @@
     <gazebo reference="left_wheel">
         <material>Gazebo/Black</material>
+    </gazebo>
+    <gazebo reference="sensor_laser">
+        <material>Gazebo/Yellow</material>
     </gazebo>
     <!--Adding Differential Drive PLugin-->
@@ -28,6 +32,38 @@
             <odometryTopic>odom</odometryTopic>
             <odometryFrame>odom</odometryFrame>
-            <robotBaseFrame>base_link</robotBaseFrame>
+            <robotBaseFrame>base_footprint</robotBaseFrame>
         </plugin>
     </gazebo>
+    <!--Laser Scanner-->
+    <gazebo reference="sensor_laser">
+    <sensor type="ray" name="head_hokuyo_sensor">
+      <pose>0 0 0 0 0 0</pose>
+      <visualize>false</visualize>
+      <update_rate>20</update_rate>
+      <ray>
+        <scan>
+          <horizontal>
+            <samples>720</samples>
+            <resolution>1</resolution>
+            <min_angle>-1.570796</min_angle>
+            <max_angle>1.570796</max_angle>
+          </horizontal>
+        </scan>
+        <range>
+          <min>0.10</min>
+          <max>10.0</max>
+          <resolution>0.01</resolution>
+        </range>
+        <noise>
+          <type>gaussian</type>
+          <mean>0.0</mean>
+          <stddev>0.01</stddev>
+        </noise>
+      </ray>
+      <plugin name="gazebo_ros_head_hokuyo_controller" filename="libgazebo_ros_laser.so">
+        <topicName>/custom_bot/laser/scan</topicName>
+        <frameName>sensor_laser</frameName>
+      </plugin>
+    </sensor>
+  </gazebo>
 </robot>

File: AMR_ws/src/custom_bot/urdf/materials.xacro (robot description, xacro)
@@ -20,3 +20,6 @@
     <color rgba="1.0 1.0 1.0 1.0"/>
   </material>
+  <material name="yellow">
+    <color rgba="1.0 1.0 0.0 1.0"/>
+  </material>
 </robot>

Commit message: Fixed collision box size to avoid laser scanner blocking

File: AMR_ws/src/custom_bot/urdf/diff_drive_bot.xacro (robot description, xacro)
@@ -40,7 +40,7 @@
         </inertial>
         <collision>
-            <origin rpy="0 0 0" xyz="0 0 0"/>
+            <origin rpy="0 0 0" xyz="0 0 -0.027"/>
             <geometry>
-                <box size="0.15 .20 .054"/>
+                <box size="0.15 .20 .045"/>
             </geometry>
         </collision>

Commit message: Add Camera

File: AMR_ws/src/custom_bot/urdf/diff_drive_bot.xacro (robot description, xacro)
@@ -12,4 +12,6 @@
     <xacro:property name="laser_radius" value="0.025"/>
     <xacro:property name="laser_height" value="0.025"/>
+    <xacro:property name="camera_dim" value="0.02 0.03 0.02"/>
+    <xacro:property name="pi_rads" value="3.14159"/>
     <!--Macros-->
     <xacro:macro name="cylinder_inertia" params="mass r l">
@@ -143,4 +145,23 @@
         </collision>
     </link>
+    <link name="sensor_camera">
+        <visual>
+            <origin rpy="0 0 0" xyz="0 0 0"/>
+            <geometry>
+                <box size="${camera_dim}"/>
+            </geometry>
+            <material name="yellow"/>
+        </visual>
+        <inertial>
+            <mass value="1"/>
+            <inertia ixx="1e-6" ixy="0" ixz="0" iyy="1e-6" iyz="0" izz="1e-6" />
+        </inertial>
+        <collision>
+            <origin rpy="0 0 0" xyz="0 0 0.0125"/>
+            <geometry>
+                <box size="${camera_dim}"/>
+            </geometry>
+        </collision>
+    </link>
     <joint name="base_foorprint_to_base_link" type="fixed">
         <origin xyz="0 0 0.0512"/>
@@ -176,3 +197,9 @@
         <child link="sensor_laser"/>
     </joint>
+    <joint name="base_link_to_camera" type="fixed">
+        <origin rpy="0 0 ${pi_rads}" xyz="-0.08 0.0 0.0"/>
+        <axis xyz="0 0 0 "/>
+        <parent link="base_link"/>
+        <child link="sensor_camera"/>
+    </joint>
 </robot>

File: AMR_ws/src/custom_bot/urdf/gazebo.xacro (robot description, xacro)
@@ -5,65 +5,103 @@
 <robot name="diff_drive_bot" xmlns:xacro="http://www.ros.org/wiki/xacro">
     <!--If the <gazebo> tag is used without reference property, it is assumed-->
-    <!--the element is for the entire robot-->
-    <!--Materials-->
-    <gazebo reference="base_link">
-        <material>Gazebo/Orange</material>
+        <!--the element is for the entire robot-->
+        <!--Materials-->
+        <gazebo reference="base_link">
+            <material>Gazebo/Orange</material>
+        </gazebo>
+        <gazebo reference="right_wheel">
+            <material>Gazebo/Black</material>
+        </gazebo>
+        <gazebo reference="left_wheel">
+            <material>Gazebo/Black</material>
+        </gazebo>
+        <gazebo reference="sensor_laser">
+            <material>Gazebo/Yellow</material>
+        </gazebo>
+        <!--Adding Differential Drive PLugin-->
+        <gazebo>
+            <plugin filename="libgazebo_ros_diff_drive.so" name="differential_drive_controller">
+                <alwaysOn>true</alwaysOn>
+                <updateRate>20</updateRate>
+                <leftJoint>base_link_to_left_wheel</leftJoint>
+                <rightJoint>base_link_to_right_wheel</rightJoint>
+                <wheelSeparation>0.4</wheelSeparation>
+                <wheelDiameter>0.2</wheelDiameter>
+                <torque>0.1</torque>
+                <commandTopic>cmd_vel</commandTopic>
+                <odometryTopic>odom</odometryTopic>
+                <odometryFrame>odom</odometryFrame>
+                <robotBaseFrame>base_footprint</robotBaseFrame>
+            </plugin>
+        </gazebo>
+        <!--Laser Scanner-->
+        <gazebo reference="sensor_laser">
+            <sensor type="ray" name="head_hokuyo_sensor">
+                <pose>0 0 0 0 0 0</pose>
+                <visualize>false</visualize>
+                <update_rate>20</update_rate>
+                <ray>
+                    <scan>
+                        <horizontal>
+                            <samples>720</samples>
+                            <resolution>1</resolution>
+                            <min_angle>-1.570796</min_angle>
+                            <max_angle>1.570796</max_angle>
+                        </horizontal>
+                    </scan>
+                    <range>
+                        <min>0.10</min>
+                        <max>10.0</max>
+                        <resolution>0.01</resolution>
+                    </range>
+                    <noise>
+                        <type>gaussian</type>
+                        <mean>0.0</mean>
+                        <stddev>0.01</stddev>
+                    </noise>
+                </ray>
+                <plugin name="gazebo_ros_head_hokuyo_controller" filename="libgazebo_ros_laser.so">
+                    <topicName>/custom_bot/laser/scan</topicName>
+                    <frameName>sensor_laser</frameName>
+                </plugin>
+            </sensor>
+        </gazebo>
+    <!--Camera-->
+    <!--Ref: http://gazebosim.org/tutorials?tut=ros_gzplugins#Camera-->
+    <gazebo reference="sensor_camera">
+        <sensor type="camera" name="camera_front">
+            <update_rate>30.0</update_rate>
+            <camera name="head">
+                <horizontal_fov>1.3962634</horizontal_fov>
+                <image>
+                    <width>800</width>
+                    <height>800</height>
+                    <format>R8G8B8</format>
+                </image>
+                <clip>
+                    <near>0.02</near>
+                    <far>300</far>
+                </clip>
+                <noise>
+                    <type>gaussian</type>
+                    <mean>0.0</mean>
+                    <stddev>0.007</stddev>
+                </noise>
+            </camera>
+            <plugin name="camera_controller" filename="libgazebo_ros_camera.so">
+                <alwaysOn>true</alwaysOn>
+                <updateRate>0.0</updateRate>
+                <cameraName>custom_bot/camera_front</cameraName>
+                <imageTopicName>image_raw</imageTopicName>
+                <cameraInfoTopicName>camera_info</cameraInfoTopicName>
+                <frameName>sensor_camera</frameName>
+                <hackBaseline>0.07</hackBaseline>
+                <distortionK1>0.0</distortionK1>
+                <distortionK2>0.0</distortionK2>
+                <distortionK3>0.0</distortionK3>
+                <distortionT1>0.0</distortionT1>
+                <distortionT2>0.0</distortionT2>
+            </plugin>
+        </sensor>
     </gazebo>
-    <gazebo reference="right_wheel">
-        <material>Gazebo/Black</material>
-    </gazebo>
-    <gazebo reference="left_wheel">
-        <material>Gazebo/Black</material>
-    </gazebo>
-    <gazebo reference="sensor_laser">
-        <material>Gazebo/Yellow</material>
-    </gazebo>
-    <!--Adding Differential Drive PLugin-->
-    <gazebo>
-        <plugin filename="libgazebo_ros_diff_drive.so" name="differential_drive_controller">
-            <alwaysOn>true</alwaysOn>
-            <updateRate>20</updateRate>
-            <leftJoint>base_link_to_left_wheel</leftJoint>
-            <rightJoint>base_link_to_right_wheel</rightJoint>
-            <wheelSeparation>0.4</wheelSeparation>
-            <wheelDiameter>0.2</wheelDiameter>
-            <torque>0.1</torque>
-            <commandTopic>cmd_vel</commandTopic>
-            <odometryTopic>odom</odometryTopic>
-            <odometryFrame>odom</odometryFrame>
-            <robotBaseFrame>base_footprint</robotBaseFrame>
-        </plugin>
-    </gazebo>
-    <!--Laser Scanner-->
-    <gazebo reference="sensor_laser">
-    <sensor type="ray" name="head_hokuyo_sensor">
-      <pose>0 0 0 0 0 0</pose>
-      <visualize>false</visualize>
-      <update_rate>20</update_rate>
-      <ray>
-        <scan>
-          <horizontal>
-            <samples>720</samples>
-            <resolution>1</resolution>
-            <min_angle>-1.570796</min_angle>
-            <max_angle>1.570796</max_angle>
-          </horizontal>
-        </scan>
-        <range>
-          <min>0.10</min>
-          <max>10.0</max>
-          <resolution>0.01</resolution>
-        </range>
-        <noise>
-          <type>gaussian</type>
-          <mean>0.0</mean>
-          <stddev>0.01</stddev>
-        </noise>
-      </ray>
-      <plugin name="gazebo_ros_head_hokuyo_controller" filename="libgazebo_ros_laser.so">
-        <topicName>/custom_bot/laser/scan</topicName>
-        <frameName>sensor_laser</frameName>
-      </plugin>
-    </sensor>
-  </gazebo>
-</robot>
+    </robot>

Commit message: Move Base

File: AMR_ws/src/custom_bot/urdf/diff_drive_bot.xacro (robot description, xacro)
@@ -180,11 +180,11 @@
     </joint>
     <joint name="base_link_to_right_wheel" type="continuous">
+        <origin rpy="-1.57079632679 0  0 " xyz="0.0267 -0.13 -0.02"/>
+        <axis xyz="0 0 1 "/>
+        <parent link="base_link"/>
+        <child link="right_wheel"/>
+    </joint>
+    <joint name="base_link_to_left_wheel" type="continuous">
         <origin rpy="1.57079632679 0  0 " xyz="0.0267 0.13 -0.02"/>
-        <axis xyz="0 0 1 "/>
-        <parent link="base_link"/>
-        <child link="right_wheel"/>
-    </joint>
-    <joint name="base_link_to_left_wheel" type="continuous">
-        <origin rpy="-1.57079632679 0  0 " xyz="0.0267 -0.13 -0.02"/>
         <axis xyz="0 0 -1 "/>
         <parent link="base_link"/>
@@ -198,5 +198,5 @@
     </joint>
     <joint name="base_link_to_camera" type="fixed">
-        <origin rpy="0 0 ${pi_rads}" xyz="-0.08 0.0 0.0"/>
+        <origin rpy="0 0 -${pi_rads}" xyz="0.08 0.0 0.0"/>
         <axis xyz="0 0 0 "/>
         <parent link="base_link"/>

Commit message: Fix camera view

File: AMR_ws/src/custom_bot/urdf/diff_drive_bot.xacro (robot description, xacro)
@@ -198,5 +198,5 @@
     </joint>
     <joint name="base_link_to_camera" type="fixed">
-        <origin rpy="0 0 -${pi_rads}" xyz="0.08 0.0 0.0"/>
+        <origin rpy="0 0 ${pi_rads}" xyz="0.08 0.0 0.0"/>
         <axis xyz="0 0 0 "/>
         <parent link="base_link"/>

Commit message: Fix Camera

File: AMR_ws/src/custom_bot/urdf/diff_drive_bot.xacro (robot description, xacro)
@@ -198,5 +198,5 @@
     </joint>
     <joint name="base_link_to_camera" type="fixed">
-        <origin rpy="0 0 ${pi_rads}" xyz="0.08 0.0 0.0"/>
+        <origin rpy="0 0 0" xyz="0.08 0.0 0.0"/>
         <axis xyz="0 0 0 "/>
         <parent link="base_link"/>
